File: pcb/icetube.brd (EAGLE design)
At the start: 142.3 x 26.9 mm, 41 parts, among them IC1 ATMEGA328P, IC2 MAX6921, IC3 7805T, J1 2.1MMJACKTHM, Q1 32.768 khz, Q2 IRFD110, Q4 PFET-ZVP2110A, SW1 ALARM

Commit message: Board and schematic as uploaded to OSH Park, by their upload board feature.
Parts:
- moved D1 0.25 mm to (11.5, 12.6)
Connections:
- net N$39: now also Q4.3; no longer Q4.S
- net VCC: now also Q4.1; no longer Q4.D
- net VFDPWR: now also Q4.2; no longer Q4.G
Other:
- board text added: "Ice Tube V1 by PhilD13"
- board text added: "based on ladyada.net"
- board text removed: "Ice Tube"
- board text removed: "ladyada.net"
